Commit message: drive base

File: models/excvModel.xacro (robot description, xacro)
@@ -2,21 +2,16 @@
 <robot name="transportation" xmlns:xacro="http://www.ros.org/wiki/xacro">
 <xacro:property name="wheel_height" value="-0.05"/>
-<xacro:property name="wheel_inertia_ixx" value="0.025"/>
-<xacro:property name="wheel_inertia_iyy" value="0.025"/>
-<xacro:property name="wheel_inertia_izz" value="0.025"/>
+<xacro:property name="wheel_length" value="0.05"/>
+<xacro:property name="wheel_offset" value="0.11"/>
+<xacro:property name="chassis_width" value="0.2"/>
+<xacro:property name="chassis_length" value="0.4"/>
 <!--Shape Macros=======================================-->
 <!--Wheel-->
 <xacro:macro name="wheel" params="name">
 <link name="${name}">
-    <collision name="${name}_collision">
+    <visual>
       <origin xyz="0 0 0" rpy="0 1.5707 1.5707"/>
       <geometry>
-        <cylinder radius="0.1" length="0.05"/>
-      </geometry>
-    </collision>
-    <visual name="${name}_wheel_visual">
-      <origin xyz="0 0 0" rpy="0 1.5707 1.5707"/>
-      <geometry>
-        <cylinder radius="0.1" length="0.05"/>
+        <cylinder radius="0.1" length="${wheel_length}"/>
       </geometry>
       <material name="black">
@@ -24,47 +19,35 @@
       </material>
     </visual>
-    <inertial>
-      <origin xyz="0 0 0" rpy="0 1.5707 1.5707"/>
-      <mass value="5"/>
-      <cylinder_inertia m="5" r="0.1" h="0.05"/>
-      <inertia
-        ixx="${wheel_inertia_ixx}" ixy="0.0" ixz="0.0"
-        iyy="${wheel_inertia_iyy}" iyz="0.0"
-        izz="${wheel_inertia_izz}"/>
-    </inertial>
   </link>
 </xacro:macro>
-<!--Robot Definition-->
-<link name='base_link'>
-    <pose>0 0 0 0 0 0</pose>
-    <inertial>
-      <mass value="20.0"/>
-      <origin xyz="0.0 0.0 0.0" rpy="0.0 0.0 0.0"/>
-      <inertia
-          ixx="0.4" ixy="0" ixz="0"
-          iyy="0.2" iyz="0"
-          izz="0.15"
-      />
-    </inertial>
-    <collision name='collision'>
-      <geometry>
-        <box size=".4 .2 .15"/>
-      </geometry>
-    </collision>
-    <visual name='base_link_visual'>
+<!--Joint Macros========================================-->
+<!--Wheel Joint-->
+<xacro:macro name="wheel_Joint" params="name parent child z_pos mirror">
+  <joint type="continuous" name="${name}_axle">
+    <origin  xyz="${z_pos} ${((chassis_width/2)+wheel_length)*mirror} ${wheel_height}" rpy="0 0 0"/>
+    <child link="${child}"/>
+    <parent link="${parent}"/>
+    <axis xyz="0 1 0" rpy="0 0 0"/>
+  </joint>
+</xacro:macro>
+<!--Robot Definition====================================-->
+<link name='chassis'>
+    <visual>
       <origin xyz="0 0 0" rpy="0 0 0"/>
       <geometry>
-        <box size=".4 .2 .15"/>
+        <box size="${chassis_length} ${chassis_width} .15"/>
       </geometry>
+      <material name="black">
+        <color rgba="0 0 0 0"/>
+      </material>
     </visual>
   </link>
-  <wheel name="frontLeftWheel" />
-  <joint type="continuous" name="left_wheel_axle">
-    <origin  xyz="0.11 0.15 ${wheel_height}" rpy="0 0 0"/>
-    <child link="frontLeftWheel"/>
-    <parent link="base_link"/>
-    <axis xyz="0 1 0" rpy="0 0 0"/>
-    <limit effort="100" velocity="100"/>
-    <joint_properties damping="0.0" friction="0.0"/>
-  </joint>
+  <wheel name="front_left" />
+  <wheel name="front_right" />
+  <wheel name="back_left" />
+  <wheel name="back_right" />
+  <wheel_Joint name="front_left" parent="chassis" child="front_left" z_pos="${wheel_offset}" mirror="1"/>
+  <wheel_Joint name="front_right" parent="chassis" child="front_right" z_pos="${wheel_offset}" mirror="-1"/>
+  <wheel_Joint name="back_left" parent="chassis" child="back_left" z_pos="${wheel_offset*-1}" mirror="1"/>
+  <wheel_Joint name="back_right" parent="chassis" child="back_right" z_pos="${wheel_offset*-1}" mirror="-1"/>
 </robot>

Commit message: added trencher

File: models/excvModel.xacro (robot description, xacro)
@@ -6,6 +6,17 @@
 <xacro:property name="chassis_width" value="0.2"/>
 <xacro:property name="chassis_length" value="0.4"/>
+<xacro:property name="chassis_height" value="0.15"/>
+<xacro:property name="chassis_cutout_length" value="0.1"/>
+<xacro:property name="chassis_cutout_width" value="0.05"/>
+<xacro:property name="trencher_mount_height" value="0.1"/>
+<xacro:property name="trencher_outer_length" value="0.3"/>
+<xacro:property name="trencher_inner_length" value="0.3"/>
+<xacro:property name="trencher_outer_width" value="${chassis_width-(chassis_cutout_width*2)}"/>
+<xacro:property name="trencher_inner_width" value="${chassis_width-(chassis_cutout_width*2)-0.025}"/>
+<xacro:property name="trencher_height" value="0.05"/>
+<!--Color Macros=======================================-->
+<xacro:property name="grey" value="0.7 0.7 0.7 1"/>
+<xacro:property name="blue" value="0 0.3 0.8 1"/>
 <!--Shape Macros=======================================-->
-<!--Wheel-->
 <xacro:macro name="wheel" params="name">
 <link name="${name}">
@@ -15,6 +26,6 @@
         <cylinder radius="0.1" length="${wheel_length}"/>
       </geometry>
-      <material name="black">
-        <color rgba="0 0 0 0"/>
+      <material name="wheel_color">
+        <color rgba="${blue}"/>
       </material>
     </visual>
@@ -22,8 +33,7 @@
 </xacro:macro>
 <!--Joint Macros========================================-->
-<!--Wheel Joint-->
-<xacro:macro name="wheel_Joint" params="name parent child z_pos mirror">
+<xacro:macro name="wheel_Joint" params="name parent child x_pos mirror">
   <joint type="continuous" name="${name}_axle">
-    <origin  xyz="${z_pos} ${((chassis_width/2)+wheel_length)*mirror} ${wheel_height}" rpy="0 0 0"/>
+    <origin  xyz="${x_pos} ${((chassis_width/2)+(wheel_length/2))*mirror} ${wheel_height}" rpy="0 0 0"/>
     <child link="${child}"/>
     <parent link="${parent}"/>
@@ -36,8 +46,52 @@
       <origin xyz="0 0 0" rpy="0 0 0"/>
       <geometry>
-        <box size="${chassis_length} ${chassis_width} .15"/>
+        <box size="${chassis_length} ${chassis_width} ${chassis_height}"/>
       </geometry>
-      <material name="black">
-        <color rgba="0 0 0 0"/>
+      <material name="chassis_color">
+        <color rgba="${grey}"/>
+      </material>
+    </visual>
+  </link>
+  <link name='left_cutout'>
+    <visual>
+      <origin xyz="0 0 ${trencher_mount_height/2}" rpy="0 0 0"/>
+      <geometry>
+        <box size="${chassis_cutout_length} ${chassis_cutout_width} ${chassis_height+trencher_mount_height}"/>
+      </geometry>
+      <material name="left_cutout_color">
+        <color rgba="${grey}"/>
+      </material>
+    </visual>
+  </link>
+  <link name='right_cutout'>
+    <visual>
+      <origin xyz="0 0 ${trencher_mount_height/2}" rpy="0 0 0"/>
+      <geometry>
+        <box size="${chassis_cutout_length} ${chassis_cutout_width} ${chassis_height+trencher_mount_height}"/>
+      </geometry>
+      <material name="right_cutout_color">
+        <color rgba="${grey}"/>
+      </material>
+    </visual>
+  </link>
+  <link name='trencher_outer'>
+    <visual>
+      <origin xyz="${trencher_outer_length/2} 0 0" rpy="0 0 0"/>
+      <geometry>
+        <box size="${trencher_outer_length} ${trencher_outer_width} ${trencher_height}"/>
+      </geometry>
+      <material name="chassis_color">
+        <color rgba="${grey}"/>
+      </material>
+    </visual>
+  </link>
+  <link name='trencher_inner'>
+    <visual>
+      <origin xyz="${trencher_inner_length/2} 0 0" rpy="0 0 0"/>
+      <geometry>
+        <box size="${trencher_inner_length} ${trencher_inner_width} ${trencher_height}"/>
+      </geometry>
+      <material name="chassis_color">
+        <color rgba="${grey}"/>
       </material>
     </visual>
@@ -47,7 +101,31 @@
   <xacro:wheel name="back_left" />
   <xacro:wheel name="back_right" />
-  <xacro:wheel_Joint name="front_left" parent="chassis" child="front_left" z_pos="${wheel_offset}" mirror="1"/>
-  <xacro:wheel_Joint name="front_right" parent="chassis" child="front_right" z_pos="${wheel_offset}" mirror="-1"/>
-  <xacro:wheel_Joint name="back_left" parent="chassis" child="back_left" z_pos="${wheel_offset*-1}" mirror="1"/>
-  <xacro:wheel_Joint name="back_right" parent="chassis" child="back_right" z_pos="${wheel_offset*-1}" mirror="-1"/>
+  <xacro:wheel_Joint name="front_left" parent="chassis" child="front_left" x_pos="${wheel_offset+(chassis_cutout_length/2)}" mirror="1"/>
+  <xacro:wheel_Joint name="front_right" parent="chassis" child="front_right" x_pos="${wheel_offset+(chassis_cutout_length/2)}" mirror="-1"/>
+  <xacro:wheel_Joint name="back_left" parent="chassis" child="back_left" x_pos="${wheel_offset*-1}" mirror="1"/>
+  <xacro:wheel_Joint name="back_right" parent="chassis" child="back_right" x_pos="${wheel_offset*-1}" mirror="-1"/>
+  <joint type="fixed" name="left_cutout_fixed">
+    <origin xyz="${(chassis_length/2)+(chassis_cutout_length/2)} ${(chassis_width/2)-(chassis_cutout_width/2)} 0" rpy="0 0 0"/>
+    <child link="left_cutout"/>
+    <parent link="chassis"/>
+  </joint>
+  <joint type="fixed" name="right_cutout_fixed">
+    <origin xyz="${(chassis_length/2)+(chassis_cutout_length/2)} ${((chassis_width/2)-(chassis_cutout_width/2))*-1} 0" rpy="0 0 0"/>
+    <child link="right_cutout"/>
+    <parent link="chassis"/>
+  </joint>
+  <joint type="revolute" name="trencher_axle">
+    <origin  xyz="0 ${chassis_cutout_width*-1.5} ${trencher_mount_height+trencher_height}" rpy="0 0 0"/>
+    <child link="trencher_outer"/>
+    <parent link="left_cutout"/>
+    <axis xyz="0 1 0" rpy="0 0 0"/>
+    <limit upper="1" lower="-2.75" effort="0" velocity="1"/>
+  </joint>
+  <joint type="prismatic" name="trencher_extend">
+    <origin  xyz="0 0 0" rpy="0 0 0"/>
+    <child link="trencher_inner"/>
+    <parent link="trencher_outer"/>
+    <axis xyz="1 0 0" rpy="0 0 0"/>
+    <limit upper="${trencher_inner_length}" lower="0" effort="0" velocity="1"/>
+  </joint>
 </robot>

Commit message: colors

File: models/excvModel.xacro (robot description, xacro)
@@ -1,4 +1,5 @@
 <?xml version='1.0' encoding="UTF-8"?>
-<robot name="transportation" xmlns:xacro="http://www.ros.org/wiki/xacro">
+<robot name="excavation" xmlns:xacro="http://www.ros.org/wiki/xacro">
+<!--Dimension Macros=====================================-->
 <xacro:property name="wheel_height" value="-0.05"/>
 <xacro:property name="wheel_length" value="0.05"/>
@@ -15,8 +16,9 @@
 <xacro:property name="trencher_inner_width" value="${chassis_width-(chassis_cutout_width*2)-0.025}"/>
 <xacro:property name="trencher_height" value="0.05"/>
-<!--Color Macros=======================================-->
+<!--Color Macros========================================-->
+<xacro:property name="dark_grey" value="0.5 0.5 0.5 1"/>
 <xacro:property name="grey" value="0.7 0.7 0.7 1"/>
 <xacro:property name="blue" value="0 0.3 0.8 1"/>
-<!--Shape Macros=======================================-->
+<!--Shape Macros========================================-->
 <xacro:macro name="wheel" params="name">
 <link name="${name}">
@@ -27,4 +29,5 @@
       </geometry>
       <material name="wheel_color">
+        <!--texture filename="file://$(find robot-model)/models/wheel_texture.jpeg"/-->
         <color rgba="${blue}"/>
       </material>
@@ -81,6 +84,6 @@
         <box size="${trencher_outer_length} ${trencher_outer_width} ${trencher_height}"/>
       </geometry>
-      <material name="chassis_color">
-        <color rgba="${grey}"/>
+      <material name="trencher_outer_color">
+        <color rgba="${dark_grey}"/>
       </material>
     </visual>
@@ -92,9 +95,10 @@
         <box size="${trencher_inner_length} ${trencher_inner_width} ${trencher_height}"/>
       </geometry>
-      <material name="chassis_color">
+      <material name="trencher_inner_color">
         <color rgba="${grey}"/>
       </material>
     </visual>
   </link>
+<!--Joints=========================================-->
   <xacro:wheel name="front_left" />
   <xacro:wheel name="front_right" />

Commit message: added wheel mesh

File: models/excvModel.xacro (robot description, xacro)
@@ -4,16 +4,19 @@
 <xacro:property name="wheel_height" value="-0.05"/>
 <xacro:property name="wheel_length" value="0.05"/>
+<xacro:property name="wheel_scale" value="0.004"/>
+<xacro:property name="wheel_mount_width" value="0.05"/>
 <xacro:property name="wheel_offset" value="0.11"/>
 <xacro:property name="chassis_width" value="0.2"/>
 <xacro:property name="chassis_length" value="0.4"/>
-<xacro:property name="chassis_height" value="0.15"/>
+<xacro:property name="chassis_height" value="0.05"/>
 <xacro:property name="chassis_cutout_length" value="0.1"/>
 <xacro:property name="chassis_cutout_width" value="0.05"/>
 <xacro:property name="trencher_mount_height" value="0.1"/>
 <xacro:property name="trencher_outer_length" value="0.3"/>
+<xacro:property name="trencher_outer_width" value="${chassis_width-(chassis_cutout_width*2)}"/>
+<xacro:property name="trencher_outer_height" value="0.05"/>
 <xacro:property name="trencher_inner_length" value="0.3"/>
-<xacro:property name="trencher_outer_width" value="${chassis_width-(chassis_cutout_width*2)}"/>
 <xacro:property name="trencher_inner_width" value="${chassis_width-(chassis_cutout_width*2)-0.025}"/>
-<xacro:property name="trencher_height" value="0.05"/>
+<xacro:property name="trencher_inner_height" value="0.045"/>
 <!--Color Macros========================================-->
 <xacro:property name="dark_grey" value="0.5 0.5 0.5 1"/>
@@ -21,14 +24,27 @@
 <xacro:property name="blue" value="0 0.3 0.8 1"/>
 <!--Shape Macros========================================-->
-<xacro:macro name="wheel" params="name">
+<xacro:macro name="wheel" params="name mirror">
 <link name="${name}">
     <visual>
-      <origin xyz="0 0 0" rpy="0 1.5707 1.5707"/>
+      <origin xyz="0 0 0" rpy="0 1.5707 ${mirror*1.5707}"/>
       <geometry>
-        <cylinder radius="0.1" length="${wheel_length}"/>
+        <!--cylinder radius="0.1" length="${wheel_length}"/-->
+          <mesh filename="file://$(find robot-model)/models/meshes/wheel.stl" scale="${wheel_scale} ${wheel_scale} ${wheel_scale}"/>
       </geometry>
       <material name="wheel_color">
-        <!--texture filename="file://$(find robot-model)/models/wheel_texture.jpeg"/-->
         <color rgba="${blue}"/>
+      </material>
+    </visual>
+  </link>
+</xacro:macro>
+<xacro:macro name="wheel_mount" params="name">
+<link name="${name}">
+    <visual>
+      <origin xyz="0 0 0" rpy="0 0 0"/>
+      <geometry>
+        <box size="${wheel_mount_width} ${wheel_mount_width} ${wheel_height}"/>
+      </geometry>
+      <material name="wheel_mount_color">
+        <color rgba="${grey}"/>
       </material>
     </visual>
@@ -38,8 +54,15 @@
 <xacro:macro name="wheel_Joint" params="name parent child x_pos mirror">
   <joint type="continuous" name="${name}_axle">
-    <origin  xyz="${x_pos} ${((chassis_width/2)+(wheel_length/2))*mirror} ${wheel_height}" rpy="0 0 0"/>
+    <origin  xyz="${x_pos} ${((chassis_width/2)+(wheel_length/2)+0.01)*mirror} ${wheel_height}" rpy="0 0 0"/>
     <child link="${child}"/>
     <parent link="${parent}"/>
     <axis xyz="0 1 0" rpy="0 0 0"/>
+  </joint>
+</xacro:macro>
+<xacro:macro name="wheel_mount_fixed" params=" name child x_pos mirror">
+  <joint type="fixed" name="${name}">
+    <origin xyz="${x_pos} ${((chassis_width/2)-(wheel_mount_width/2))*mirror} ${wheel_height}" rpy="0 0 0"/>
+    <child link="${child}"/>
+    <parent link="chassis"/>
   </joint>
 </xacro:macro>
@@ -82,5 +105,5 @@
       <origin xyz="${trencher_outer_length/2} 0 0" rpy="0 0 0"/>
       <geometry>
-        <box size="${trencher_outer_length} ${trencher_outer_width} ${trencher_height}"/>
+        <box size="${trencher_outer_length} ${trencher_outer_width} ${trencher_outer_height}"/>
       </geometry>
       <material name="trencher_outer_color">
@@ -93,5 +116,5 @@
       <origin xyz="${trencher_inner_length/2} 0 0" rpy="0 0 0"/>
       <geometry>
-        <box size="${trencher_inner_length} ${trencher_inner_width} ${trencher_height}"/>
+        <box size="${trencher_inner_length} ${trencher_inner_width} ${trencher_inner_height}"/>
       </geometry>
       <material name="trencher_inner_color">
@@ -101,12 +124,20 @@
   </link>
 <!--Joints=========================================-->
-  <xacro:wheel name="front_left" />
-  <xacro:wheel name="front_right" />
-  <xacro:wheel name="back_left" />
-  <xacro:wheel name="back_right" />
+  <xacro:wheel name="front_left" mirror="-1"/>
+  <xacro:wheel name="front_right" mirror="1"/>
+  <xacro:wheel name="back_left" mirror="-1"/>
+  <xacro:wheel name="back_right" mirror="1"/>
+  <xacro:wheel_mount name="front_left_mount" />
+  <xacro:wheel_mount name="front_right_mount" />
+  <xacro:wheel_mount name="back_left_mount" />
+  <xacro:wheel_mount name="back_right_mount" />
   <xacro:wheel_Joint name="front_left" parent="chassis" child="front_left" x_pos="${wheel_offset+(chassis_cutout_length/2)}" mirror="1"/>
   <xacro:wheel_Joint name="front_right" parent="chassis" child="front_right" x_pos="${wheel_offset+(chassis_cutout_length/2)}" mirror="-1"/>
   <xacro:wheel_Joint name="back_left" parent="chassis" child="back_left" x_pos="${wheel_offset*-1}" mirror="1"/>
   <xacro:wheel_Joint name="back_right" parent="chassis" child="back_right" x_pos="${wheel_offset*-1}" mirror="-1"/>
+  <xacro:wheel_mount_fixed name="front_left_fixed" child="front_left_mount" x_pos="${wheel_offset+(chassis_cutout_length/2)}" mirror="1"/>
+  <xacro:wheel_mount_fixed name="front_right_fixed" child="front_right_mount" x_pos="${wheel_offset+(chassis_cutout_length/2)}" mirror="-1"/>
+  <xacro:wheel_mount_fixed name="back_left_fixed" child="back_left_mount" x_pos="${wheel_offset*-1}" mirror="1"/>
+  <xacro:wheel_mount_fixed name="back_right_fixed" child="back_right_mount" x_pos="${wheel_offset*-1}" mirror="-1"/>
   <joint type="fixed" name="left_cutout_fixed">
     <origin xyz="${(chassis_length/2)+(chassis_cutout_length/2)} ${(chassis_width/2)-(chassis_cutout_width/2)} 0" rpy="0 0 0"/>
@@ -120,5 +151,5 @@
   </joint>
   <joint type="revolute" name="trencher_axle">
-    <origin  xyz="0 ${chassis_cutout_width*-1.5} ${trencher_mount_height+trencher_height}" rpy="0 0 0"/>
+    <origin  xyz="0 ${chassis_cutout_width*-1.5} ${(trencher_mount_height/2)+(trencher_outer_height)}" rpy="0 0 0"/>
     <child link="trencher_outer"/>
     <parent link="left_cutout"/>
