Commit message: added Hopper

File: models/excvModelSimple.xacro (robot description, xacro)
@@ -1,4 +1,4 @@
 <?xml version='1.0' encoding="UTF-8"?>
-<robot name="excavation" xmlns:xacro="http://www.ros.org/wiki/xacro">
+<robot name="excavation_simple" xmlns:xacro="http://www.ros.org/wiki/xacro">
 <!--Dimension Macros=====================================-->
 <xacro:property name="wheel_height" value="-0.05"/>
@@ -19,4 +19,9 @@
 <xacro:property name="trencher_inner_width" value="${chassis_width-(chassis_cutout_width*2)-0.025}"/>
 <xacro:property name="trencher_inner_height" value="0.045"/>
+<xacro:property name="hopper_length" value="0.1"/>
+<xacro:property name="hopper_width" value="0.15"/>
+<xacro:property name="hopper_height" value="0.1"/>
+<xacro:property name="hopper_mount_height" value="0.15"/>
+<xacro:property name="hopper_mount_size" value="0.05"/>
 <!--Color Macros========================================-->
 <xacro:property name="dark_grey" value="0.5 0.5 0.5 1"/>
@@ -29,6 +34,6 @@
       <origin xyz="0 0 0" rpy="0 1.5707 ${mirror*1.5707}"/>
       <geometry>
-        <!--cylinder radius="0.1" length="${wheel_length}"/-->
-          <mesh filename="file://$(find robot-model)/models/meshes/wheel.stl" scale="${wheel_scale} ${wheel_scale} ${wheel_scale}"/>
+        <cylinder radius="0.1" length="${wheel_length}"/>
+          <!--mesh filename="file://$(find robot-model)/models/meshes/wheel.stl" scale="${wheel_scale} ${wheel_scale} ${wheel_scale}"/-->
       </geometry>
       <material name="wheel_color">
@@ -46,4 +51,17 @@
       </geometry>
       <material name="wheel_mount_color">
+        <color rgba="${grey}"/>
+      </material>
+    </visual>
+  </link>
+</xacro:macro>
+<xacro:macro name="hopper_mount" params="name">
+  <link name="${name}_hopper_mount">
+    <visual>
+      <origin xyz="0 0 0" rpy="0 0 0"/>
+      <geometry>
+        <box size="${hopper_mount_size} ${hopper_mount_size} ${hopper_mount_height+(hopper_height/2)}"/>
+      </geometry>
+      <material name="${name}_hopper_mount_color">
         <color rgba="${grey}"/>
       </material>
@@ -54,5 +72,5 @@
 <xacro:macro name="wheel_Joint" params="name parent child x_pos mirror">
   <joint type="continuous" name="${name}_axle">
-    <origin  xyz="${x_pos} ${((chassis_width/2)+(wheel_length/2)+0.01)*mirror} ${wheel_height}" rpy="0 0 0"/>
+    <origin  xyz="${x_pos} ${((chassis_width/2)+(wheel_length/2))*mirror} ${wheel_height}" rpy="0 0 0"/>
     <child link="${child}"/>
     <parent link="${parent}"/>
@@ -60,5 +78,5 @@
   </joint>
 </xacro:macro>
-<xacro:macro name="wheel_mount_fixed" params=" name child x_pos mirror">
+<xacro:macro name="wheel_mount_fixed" params="name child x_pos mirror">
   <joint type="fixed" name="${name}">
     <origin xyz="${x_pos} ${((chassis_width/2)-(wheel_mount_width/2))*mirror} ${wheel_height}" rpy="0 0 0"/>
@@ -67,4 +85,23 @@
   </joint>
 </xacro:macro>
+<xacro:macro name="hopper_mount_fixed" params="name child x_pos mirror">
+  <joint type="fixed" name="${name}_hopper_mount_fixed">
+    <origin xyz="${x_pos} ${((chassis_width/2)-(hopper_mount_size/2))*mirror} ${(chassis_height/2)+(hopper_mount_height/2)}" rpy="0 0 0"/>
+    <child link="${child}"/>
+    <parent link="chassis"/>
+  </joint>
+</xacro:macro>
+<!--Transmission Macros========================================-->
+<xacro:macro name="wheel_transmission" params="name joint">
+  <transmission name="${name}_transmission">
+    <type>transmission_interface/SimpleTransmission</type>
+    <joint name="${joint}">
+      <hardwareInterface>hardware_interface/VelocityJointInterface</hardwareInterface>
+    </joint>
+    <actuator name="${name}_motor">
+      <hardwareInterface>hardware_interface/VelocityJointInterface</hardwareInterface>
+    </actuator>
+  </transmission>
+</xacro:macro>
 <!--Robot Definition====================================-->
 <link name='chassis'>
@@ -123,9 +160,22 @@
     </visual>
   </link>
-<!--Joints=========================================-->
+<link name='hopper'>
+    <visual>
+      <origin xyz="0 0 0" rpy="0 0 0"/>
+      <geometry>
+        <box size="${hopper_length} ${hopper_width} ${hopper_height}"/>
+      </geometry>
+      <material name="hopper_color">
+        <color rgba="${blue}"/>
+      </material>
+    </visual>
+  </link>
   <xacro:wheel name="front_left" mirror="-1"/>
   <xacro:wheel name="front_right" mirror="1"/>
   <xacro:wheel name="back_left" mirror="-1"/>
   <xacro:wheel name="back_right" mirror="1"/>
+  <xacro:hopper_mount name="left" />
+  <xacro:hopper_mount name="right" />
+<!--Joints=========================================-->
   <xacro:wheel_mount name="front_left_mount" />
   <xacro:wheel_mount name="front_right_mount" />
@@ -140,4 +190,6 @@
   <xacro:wheel_mount_fixed name="back_left_fixed" child="back_left_mount" x_pos="${wheel_offset*-1}" mirror="1"/>
   <xacro:wheel_mount_fixed name="back_right_fixed" child="back_right_mount" x_pos="${wheel_offset*-1}" mirror="-1"/>
+  <xacro:hopper_mount_fixed name="left" child="left_hopper_mount" x_pos="${(chassis_length/-2)+(hopper_mount_size/2)}" mirror="1"/>
+  <xacro:hopper_mount_fixed name="right" child="right_hopper_mount" x_pos="${(chassis_length/-2)+(hopper_mount_size/2)}" mirror="-1"/>
   <joint type="fixed" name="left_cutout_fixed">
     <origin xyz="${(chassis_length/2)+(chassis_cutout_length/2)} ${(chassis_width/2)-(chassis_cutout_width/2)} 0" rpy="0 0 0"/>
@@ -164,3 +216,10 @@
     <limit upper="${trencher_inner_length}" lower="0" effort="0" velocity="1"/>
   </joint>
+  <joint type="fixed" name="hopper_cutout_fixed">
+    <origin xyz="${(chassis_length/-2)+(hopper_length/-2)} ${(chassis_width/2)-(hopper_width/2)} ${hopper_mount_height}" rpy="0 0 0"/>
+    <child link="hopper"/>
+    <parent link="chassis"/>
+  </joint>
+<!--Transmissions=========================================-->
+  <xacro:wheel_transmission name="front_left" joint="front_left_axle"/>
 </robot>

Commit message: added model comments

File: models/excvModelSimple.xacro (robot description, xacro)
@@ -1,4 +1,8 @@
 <?xml version='1.0' encoding="UTF-8"?>
 <robot name="excavation_simple" xmlns:xacro="http://www.ros.org/wiki/xacro">
+<!--Macros-->
+<!--  Macros are constants that can be used to define any
+      aspect of the model.  They can define things like
+      values, colors, links, joints, transmissions, ect.-->
 <!--Dimension Macros=====================================-->
 <xacro:property name="wheel_height" value="-0.05"/>
@@ -94,5 +98,5 @@
 <!--Transmission Macros========================================-->
 <xacro:macro name="wheel_transmission" params="name joint">
-  <transmission name="${name}_transmission">
+  <transmission name="${name}_wheel_transmission">
     <type>transmission_interface/SimpleTransmission</type>
     <joint name="${joint}">
@@ -104,5 +108,9 @@
   </transmission>
 </xacro:macro>
-<!--Robot Definition====================================-->
+<!--Links====================================-->
+<!--  Links are the physical pieces of the model.  They
+      can be defined to have diffenet shapes, sizes, and
+      materials.  Meshes can be used to give links a
+      completly custom appearance-->
 <link name='chassis'>
     <visual>
@@ -178,4 +186,7 @@
   <xacro:hopper_mount name="right" />
 <!--Joints=========================================-->
+<!--  Joints connect links together.  Joints can be
+      of different types that dictate the type of
+      motion they have-->
   <xacro:wheel_mount name="front_left_mount" />
   <xacro:wheel_mount name="front_right_mount" />
@@ -222,4 +233,18 @@
   </joint>
 <!--Transmissions=========================================-->
+<!--  Transmissions allow joints to listen for ROS messages,
+      all transmissions must be added to a yaml file-->
   <xacro:wheel_transmission name="front_left" joint="front_left_axle"/>
+  <xacro:wheel_transmission name="front_right" joint="front_right_axle"/>
+  <xacro:wheel_transmission name="back_left" joint="back_left_axle"/>
+  <xacro:wheel_transmission name="back_right" joint="back_right_axle"/>
+  <transmission name="trencher_pivot_transmission">
+    <type>transmission_interface/SimpleTransmission</type>
+    <joint name="trencher_axle">
+      <hardwareInterface>hardware_interface/VelocityJointInterface</hardwareInterface>
+    </joint>
+    <actuator name="trencher_axle_motor">
+      <hardwareInterface>hardware_interface/VelocityJointInterface</hardwareInterface>
+    </actuator>
+  </transmission>
 </robot>
